Commit message: fixed description for upsidedown true

File: schunk_description/urdf/pw70/pw70.urdf.xacro (robot description, xacro)
@@ -17,5 +17,5 @@
         <parent link="${name}_link" />
         <child link="${name}_tilt_link" />
-        <axis xyz="0 1 0" />
+        <axis xyz="1 0  0" />
         <limit effort="12.0" velocity="4.1" lower="${-4/6 * M_PI}" upper="${4/6 * M_PI}"/>
         <calibration rising="0.0"/>
@@ -29,15 +29,13 @@
           </geometry>
         </visual>
-        <!--
         <collision>
           <geometry>
-            <mesh filename="package://schunk_description/meshes/pw70/pw70_tilt.stl" />
+            <mesh filename="package://schunk_description/meshes/pw70/pw70_tilt1.stl" />
           </geometry>
         </collision>
-        -->
       </link>
       <joint name="${name}_pan_joint" type="revolute" >
         <origin xyz="0 0 0.0951" rpy="0 0 0"/>
-        <parent link="${name}_tilt_joint" />
+        <parent link="${name}_link" />
         <child link="${name}_pan_link" />
         <axis xyz="0 0 1" />
@@ -53,11 +51,9 @@
           </geometry>
         </visual>
-        <!--
         <collision>
           <geometry>
-            <mesh filename="package://schunk_description/meshes/pw70/pw70_pan.stl" />
+            <mesh filename="package://schunk_description/meshes/pw70/pw70_pan1.stl" />
           </geometry>
         </collision>
-        -->
       </link>
       <joint name="${name}_tool_joint" type="fixed" >
@@ -74,11 +70,9 @@
           </geometry>
         </visual>
-        <!--
         <collision>
           <geometry>
-            <mesh filename="package://schunk_description/meshes/pw70/pw70_base.stl" />
+            <mesh filename="package://schunk_description/meshes/pw70/pw70_base1.stl" />
           </geometry>
         </collision>
-        -->
       </link>
     </xacro:unless>
@@ -92,16 +86,14 @@
         <xacro:default_inertial/>
         <visual>
-          <origin xyz="0 0 0" rpy="0 0 0" />
+          <origin xyz="0 0 0" rpy="3.14 0 0" />
           <geometry>
-            <mesh filename="package://schunk_description/meshes/pw70/pw70_base.dae" />
+            <mesh filename="package://schunk_description/meshes/pw70/pw70_base1.stl" />
           </geometry>
         </visual>
-        <!--
         <collision>
           <geometry>
-            <mesh filename="package://schunk_description/meshes/pw70/pw70_base.stl" />
+            <mesh filename="package://schunk_description/meshes/pw70/pw70_base1.stl" />
           </geometry>
         </collision>
-        -->
       </link>
       <joint name="${name}_pan_joint" type="revolute" >
@@ -116,22 +108,20 @@
         <xacro:default_inertial/>
         <visual>
-          <origin xyz="0 0 0" rpy="0 0 0" />
+          <origin xyz="0 0 0" rpy="3.14 0 0" />
           <geometry>
-            <mesh filename="package://schunk_description/meshes/pw70/pw70_pan.dae" />
+            <mesh filename="package://schunk_description/meshes/pw70/pw70_pan1.stl" />
           </geometry>
         </visual>
-        <!--
         <collision>
           <geometry>
-            <mesh filename="package://schunk_description/meshes/pw70/pw70_pan.stl" />
+            <mesh filename="package://schunk_description/meshes/pw70/pw70_pan1.stl"/>
           </geometry>
         </collision>
-        -->
       </link>
       <joint name="${name}_tilt_joint" type="revolute" >
-        <origin xyz="0 0 0.0951" rpy="0 0 0"/>
+        <origin xyz="0 0 0.000951" rpy="0 0 0"/>
         <parent link="${name}_pan_link" />
         <child link="${name}_tilt_link" />
-        <axis xyz="0 -1 0" />
+        <axis xyz="-1 0 0" />
         <limit effort="12.0" velocity="4.1" lower="${-4/6 * M_PI}" upper="${4/6 * M_PI}"/>
         <calibration rising="0.0"/>
@@ -140,19 +130,17 @@
         <xacro:default_inertial/>
         <visual>
-          <origin xyz="0 0 0" rpy="0 0 0" />
+          <origin xyz="0 0 0" rpy="3.14 0 0" />
           <geometry>
-            <mesh filename="package://schunk_description/meshes/pw70/pw70_tilt.dae" />
+            <mesh filename="package://schunk_description/meshes/pw70/pw70_tilt1.stl" />
           </geometry>
         </visual>
-        <!--
         <collision>
           <geometry>
-            <mesh filename="package://schunk_description/meshes/pw70/pw70_tilt.stl" />
+            <mesh filename="package://schunk_description/meshes/pw70/pw70_tilt1.stl" />
           </geometry>
         </collision>
-        -->
       </link>
       <joint name="${name}_tool_joint" type="fixed" >
-        <origin xyz="0 0 0.07" rpy="0 0 0"/>
+        <origin xyz="0 0 0.0007" rpy="0 0 0"/>
         <parent link="${name}_tilt_link" />
         <child link="${name}_tool_link" />

Commit message: pw70 working

File: schunk_description/urdf/pw70/pw70.urdf.xacro (robot description, xacro)
@@ -12,4 +12,15 @@
       <link name="${name}_link">
         <xacro:default_inertial/>
+	<visual>
+          <origin xyz="0 0 0.07" rpy="0 0 0" />
+          <geometry>
+            <mesh filename="package://schunk_description/meshes/pw70/pw70_square_holder.stl" />
+          </geometry>
+        </visual>
+<!--        <collision>
+          <geometry>
+            <mesh filename="package://schunk_description/meshes/pw70/pw70_square_holder.stl" />
+          </geometry>
+        </collision>  -->
       </link>
       <joint name="${name}_tilt_joint" type="revolute" >
@@ -17,5 +28,5 @@
         <parent link="${name}_link" />
         <child link="${name}_tilt_link" />
-        <axis xyz="1 0  0" />
+        <axis xyz="-1 0  0" />
         <limit effort="12.0" velocity="4.1" lower="${-4/6 * M_PI}" upper="${4/6 * M_PI}"/>
         <calibration rising="0.0"/>
@@ -26,21 +37,21 @@
           <origin xyz="0 0 0" rpy="0 0 0" />
           <geometry>
-            <mesh filename="package://schunk_description/meshes/pw70/pw70_tilt.dae" />
+            <mesh filename="package://schunk_description/meshes/pw70/pw70_body.stl" />
           </geometry>
         </visual>
-        <collision>
+<!--        <collision>
           <geometry>
-            <mesh filename="package://schunk_description/meshes/pw70/pw70_tilt1.stl" />
+            <mesh filename="package://schunk_description/meshes/pw70/pw70_body.stl" />
           </geometry>
-        </collision>
+        </collision>-->
       </link>
       <joint name="${name}_pan_joint" type="revolute" >
-        <origin xyz="0 0 0.0951" rpy="0 0 0"/>
-        <parent link="${name}_link" />
+        <origin xyz="0 0 0" rpy="0 0 0"/>
+        <parent link="${name}_tilt_link" />
         <child link="${name}_pan_link" />
         <axis xyz="0 0 1" />
         <limit effort="200" velocity="${2 * M_PI}" lower="${-7/3 * M_PI}" upper="${7/3 * M_PI}"/>
         <calibration rising="0.0"/>
-      </joint>
+     </joint>
       <link name="${name}_pan_link">
         <xacro:default_inertial/>
@@ -48,15 +59,15 @@
           <origin xyz="0 0 0" rpy="0 0 0" />
           <geometry>
-            <mesh filename="package://schunk_description/meshes/pw70/pw70_pan.dae" />
+            <mesh filename="package://schunk_description/meshes/pw70/pw70_round_holder.stl" />
           </geometry>
         </visual>
-        <collision>
+<!--        <collision>
           <geometry>
-            <mesh filename="package://schunk_description/meshes/pw70/pw70_pan1.stl" />
+            <mesh filename="package://schunk_description/meshes/pw70/pw70_round_holder.stl" />
           </geometry>
-        </collision>
+        </collision>-->
       </link>
       <joint name="${name}_tool_joint" type="fixed" >
-        <origin xyz="0 0 0.07" rpy="0 0 0"/>
+        <origin xyz="0 0 0.095" rpy="0 0 0"/>
         <parent link="${name}_pan_link" />
         <child link="${name}_tool_link" />
@@ -64,15 +75,4 @@
       <link name="${name}_tool_link">
         <xacro:default_inertial/>
-        <visual>
-          <origin xyz="0 0 0" rpy="0 0 0" />
-          <geometry>
-            <mesh filename="package://schunk_description/meshes/pw70/pw70_base.dae" />
-          </geometry>
-        </visual>
-        <collision>
-          <geometry>
-            <mesh filename="package://schunk_description/meshes/pw70/pw70_base1.stl" />
-          </geometry>
-        </collision>
       </link>
     </xacro:unless>
@@ -86,17 +86,17 @@
         <xacro:default_inertial/>
         <visual>
-          <origin xyz="0 0 0" rpy="3.14 0 0" />
+          <origin xyz="0 0 0.095" rpy="${M_PI} 0 0" />
           <geometry>
-            <mesh filename="package://schunk_description/meshes/pw70/pw70_base1.stl" />
+            <mesh filename="package://schunk_description/meshes/pw70/pw70_round_holder.stl" />
           </geometry>
         </visual>
-        <collision>
+<!--        <collision>
           <geometry>
-            <mesh filename="package://schunk_description/meshes/pw70/pw70_base1.stl" />
+            <mesh filename="package://schunk_description/meshes/pw70/pw70_round_holder.stl" />
           </geometry>
-        </collision>
+        </collision>-->
       </link>
       <joint name="${name}_pan_joint" type="revolute" >
-        <origin xyz="0 0 0" rpy="0 0 0"/>
+        <origin xyz="0 0 0.095" rpy="0 0 0"/>
         <parent link="${name}_link" />
         <child link="${name}_pan_link" />
@@ -108,17 +108,17 @@
         <xacro:default_inertial/>
         <visual>
-          <origin xyz="0 0 0" rpy="3.14 0 0" />
+          <origin xyz="0 0 0" rpy="${M_PI} 0 0" />
           <geometry>
-            <mesh filename="package://schunk_description/meshes/pw70/pw70_pan1.stl" />
+            <mesh filename="package://schunk_description/meshes/pw70/pw70_body.stl" />
           </geometry>
         </visual>
-        <collision>
+<!--        <collision>
           <geometry>
-            <mesh filename="package://schunk_description/meshes/pw70/pw70_pan1.stl"/>
+            <mesh filename="package://schunk_description/meshes/pw70/pw70_body.stl"/>
           </geometry>
-        </collision>
+        </collision>   -->
       </link>
       <joint name="${name}_tilt_joint" type="revolute" >
-        <origin xyz="0 0 0.000951" rpy="0 0 0"/>
+        <origin xyz="0 0 0" rpy="0 0 0"/>
         <parent link="${name}_pan_link" />
         <child link="${name}_tilt_link" />
@@ -130,17 +130,17 @@
         <xacro:default_inertial/>
         <visual>
-          <origin xyz="0 0 0" rpy="3.14 0 0" />
+          <origin xyz="0 0 0" rpy="${M_PI} 0 0" />
           <geometry>
-            <mesh filename="package://schunk_description/meshes/pw70/pw70_tilt1.stl" />
+            <mesh filename="package://schunk_description/meshes/pw70/pw70_square_holder.stl" />
           </geometry>
         </visual>
-        <collision>
+        <!--<collision>
           <geometry>
-            <mesh filename="package://schunk_description/meshes/pw70/pw70_tilt1.stl" />
+            <mesh filename="package://schunk_description/meshes/pw70/pw70_square_holder.stl" />
           </geometry>
-        </collision>
+        </collision>    -->
       </link>
       <joint name="${name}_tool_joint" type="fixed" >
-        <origin xyz="0 0 0.0007" rpy="0 0 0"/>
+        <origin xyz="0 0 0.07" rpy="0 0 0"/>
         <parent link="${name}_tilt_link" />
         <child link="${name}_tool_link" />
