Commit message: Updated description of SDH to add sensor frames

File: schunk_description/urdf/sdh/sdh.urdf.xacro (robot description, xacro)
@@ -17,5 +17,5 @@
           <mesh filename="package://schunk_description/meshes/sdh/palm.stl" />
         </geometry>
-        <material name="Schunk/LightGrey" />
+        <material name="Schunk/DarkGrey" />
       </visual>
       <collision>
@@ -71,10 +71,10 @@
     <!-- joint between sdh_palm_link and sdh_finger_11_link -->
     <joint name="${name}_knuckle_joint" type="revolute">
-      <origin xyz="0.01905 0.033 0.0745" rpy="0 0 3.14159265" />
+      <origin xyz="0.01905 0.033 0.0745" rpy="0 0 ${M_PI}" />
       <parent link="${name}_palm_link"/>
       <child link="${name}_finger_11_link"/>
       <axis xyz="0 0 1" />
       <dynamics damping="1" />
-      <limit effort="100" lower="0" upper="1.570796327" velocity="5"/>
+      <limit effort="100" lower="0" upper="${M_PI/2}" velocity="5"/>
     </joint>
     <link name="${name}_finger_11_link">
@@ -85,5 +85,5 @@
           <mesh filename="package://schunk_description/meshes/sdh/knuckle.stl" />
         </geometry>
-        <material name="Schunk/LightGrey" />
+        <material name="Schunk/DarkGrey" />
       </visual>
       <collision>
@@ -101,5 +101,5 @@
       <axis xyz="0 1 0" />
       <dynamics damping="1" />
-      <limit effort="100" lower="-1.570796327" upper="1.570796327" velocity="5"/>
+      <limit effort="100" lower="${-M_PI/2}" upper="${M_PI/2}" velocity="5"/>
     </joint>
     <link name="${name}_finger_12_link">
@@ -110,12 +110,33 @@
           <mesh filename="package://schunk_description/meshes/sdh/finger.stl" />
         </geometry>
-      <material name="Schunk/LightGrey" />
-      </visual>
-      <collision>
-        <origin xyz="0 0 0" rpy="0 0 0" />
-        <geometry>
-          <mesh filename="package://schunk_description/meshes/sdh/finger.stl"/>
-        </geometry>
-      </collision>
+      <material name="Schunk/DarkGrey" />
+      </visual>
+      <collision>
+        <origin xyz="0 0 0" rpy="0 0 0" />
+        <geometry>
+          <mesh filename="package://schunk_description/meshes/sdh/finger.stl"/>
+        </geometry>
+      </collision>
+    </link>
+    <joint name="${name}_finger_1_sensor_joint" type="fixed">
+      <origin xyz="0.01529 -0.011 ${0.01875+0.05}" rpy="-${M_PI/2} 0 ${M_PI/2}" />
+      <parent link="${name}_finger_12_link"/>
+      <child link="${name}_finger_1_sensor_link"/>
+    </joint>
+    <link name="${name}_finger_1_sensor_link">
+      <xacro:default_inertial/>
+      <!--<visual>
+        <origin xyz="0 0 0" rpy="0 0 0" />
+        <geometry>
+          <mesh filename="package://schunk_description/meshes/sdh/finger.stl" />
+        </geometry>
+      <material name="Schunk/DarkGrey" />
+      </visual>
+      <collision>
+        <origin xyz="0 0 0" rpy="0 0 0" />
+        <geometry>
+          <mesh filename="package://schunk_description/meshes/sdh/finger.stl"/>
+        </geometry>
+      </collision>-->
     </link>
     <!-- joint between sdh_finger_12_link and sdh_finger_13_link -->
@@ -126,5 +147,5 @@
       <axis xyz="0 1 0" />
       <dynamics damping="1" />
-      <limit effort="100" lower="-1.570796327" upper="1.570796327" velocity="5"/>
+      <limit effort="100" lower="${-M_PI/2}" upper="${M_PI/2}" velocity="5"/>
     </joint>
     <link name="${name}_finger_13_link">
@@ -135,5 +156,5 @@
           <mesh filename="package://schunk_description/meshes/sdh/finger_tip.stl" />
         </geometry>
-        <material name="Schunk/LightGrey" />
+        <material name="Schunk/DarkGrey" />
       </visual>
       <collision>
@@ -143,4 +164,25 @@
         </geometry>
       </collision>
+    </link>
+    <joint name="${name}_finger_tip_1_sensor_joint" type="fixed">
+      <origin xyz="0.005151 -0.011 ${0.01943+0.05}" rpy="-${M_PI/2} 0 ${M_PI/2}" />
+      <parent link="${name}_finger_13_link"/>
+      <child link="${name}_finger_tip_1_sensor_link"/>
+    </joint>
+    <link name="${name}_finger_tip_1_sensor_link">
+      <xacro:default_inertial/>
+      <!--<visual>
+        <origin xyz="0 0 0" rpy="0 0 0" />
+        <geometry>
+          <mesh filename="package://schunk_description/meshes/sdh/finger.stl" />
+        </geometry>
+      <material name="Schunk/DarkGrey" />
+      </visual>
+      <collision>
+        <origin xyz="0 0 0" rpy="0 0 0" />
+        <geometry>
+          <mesh filename="package://schunk_description/meshes/sdh/finger.stl"/>
+        </geometry>
+      </collision>-->
     </link>
     <!-- finger2 -->
@@ -148,10 +190,10 @@
     <joint name="${name}_finger_21_joint" type="revolute">
       <mimic joint="${name}_knuckle_joint" multiplier="1" offset="0"/>
-      <origin xyz="0.01905 -0.033 0.0745" rpy="0 0 3.14159265" />
+      <origin xyz="0.01905 -0.033 0.0745" rpy="0 0 ${M_PI}" />
       <parent link="${name}_palm_link"/>
       <child link="${name}_finger_21_link"/>
       <axis xyz="0 0 -1" />
       <dynamics damping="1" />
-      <limit effort="100" lower="0" upper="1.570796327" velocity="5"/>
+      <limit effort="100" lower="0" upper="${M_PI/2}" velocity="5"/>
     </joint>
     <link name="${name}_finger_21_link">
@@ -162,5 +204,5 @@
           <mesh filename="package://schunk_description/meshes/sdh/knuckle.stl" />
         </geometry>
-        <material name="Schunk/LightGrey" />
+        <material name="Schunk/DarkGrey" />
       </visual>
       <collision>
@@ -178,5 +220,5 @@
       <axis xyz="0 1 0" />
       <dynamics damping="1" />
-      <limit effort="100" lower="-1.570796327" upper="1.570796327" velocity="5"/>
+      <limit effort="100" lower="${-M_PI/2}" upper="${M_PI/2}" velocity="5"/>
     </joint>
     <link name="${name}_finger_22_link">
@@ -187,12 +229,33 @@
           <mesh filename="package://schunk_description/meshes/sdh/finger.stl" />
         </geometry>
-        <material name="Schunk/LightGrey" />
-      </visual>
-      <collision>
-        <origin xyz="0 0 0" rpy="0 0 0" />
-        <geometry>
-          <mesh filename="package://schunk_description/meshes/sdh/finger.stl"/>
-        </geometry>
-      </collision>
+        <material name="Schunk/DarkGrey" />
+      </visual>
+      <collision>
+        <origin xyz="0 0 0" rpy="0 0 0" />
+        <geometry>
+          <mesh filename="package://schunk_description/meshes/sdh/finger.stl"/>
+        </geometry>
+      </collision>
+    </link>
+    <joint name="${name}_finger_2_sensor_joint" type="fixed">
+      <origin xyz="0.01529 -0.011 ${0.01875+0.05}" rpy="-${M_PI/2} 0 ${M_PI/2}" />
+      <parent link="${name}_finger_22_link"/>
+      <child link="${name}_finger_2_sensor_link"/>
+    </joint>
+    <link name="${name}_finger_2_sensor_link">
+      <xacro:default_inertial/>
+      <!--<visual>
+        <origin xyz="0 0 0" rpy="0 0 0" />
+        <geometry>
+          <mesh filename="package://schunk_description/meshes/sdh/finger.stl" />
+        </geometry>
+      <material name="Schunk/DarkGrey" />
+      </visual>
+      <collision>
+        <origin xyz="0 0 0" rpy="0 0 0" />
+        <geometry>
+          <mesh filename="package://schunk_description/meshes/sdh/finger.stl"/>
+        </geometry>
+      </collision>-->
     </link>
     <!-- joint between sdh_finger_22_link and sdh_finger_23_link -->
@@ -203,5 +266,5 @@
       <axis xyz="0 1 0" />
       <dynamics damping="1" />
-      <limit effort="100" lower="-1.570796327" upper="1.570796327" velocity="5"/>
+      <limit effort="100" lower="${-M_PI/2}" upper="${M_PI/2}" velocity="5"/>
     </joint>
     <link name="${name}_finger_23_link">
@@ -212,5 +275,5 @@
           <mesh filename="package://schunk_description/meshes/sdh/finger_tip.stl" />
         </geometry>
-        <material name="Schunk/LightGrey" />
+        <material name="Schunk/DarkGrey" />
       </visual>
       <collision>
@@ -220,4 +283,25 @@
         </geometry>
       </collision>
+    </link>
+    <joint name="${name}_finger_tip_2_sensor_joint" type="fixed">
+      <origin xyz="0.005151 -0.011 ${0.01943+0.05}" rpy="-${M_PI/2} 0 ${M_PI/2}" />
+      <parent link="${name}_finger_23_link"/>
+      <child link="${name}_finger_tip_2_sensor_link"/>
+    </joint>
+    <link name="${name}_finger_tip_2_sensor_link">
+      <xacro:default_inertial/>
+      <!--<visual>
+        <origin xyz="0 0 0" rpy="0 0 0" />
+        <geometry>
+          <mesh filename="package://schunk_description/meshes/sdh/finger.stl" />
+        </geometry>
+      <material name="Schunk/DarkGrey" />
+      </visual>
+      <collision>
+        <origin xyz="0 0 0" rpy="0 0 0" />
+        <geometry>
+          <mesh filename="package://schunk_description/meshes/sdh/finger.stl"/>
+        </geometry>
+      </collision>-->
     </link>
     <!-- thumb -->
@@ -235,5 +319,5 @@
           <mesh filename="package://schunk_description/meshes/sdh/knuckle.stl" />
         </geometry>
-        <material name="Schunk/LightGrey" />
+        <material name="Schunk/DarkGrey" />
       </visual>
       <collision>
@@ -251,5 +335,5 @@
     <axis xyz="0 1 0" />
     <dynamics damping="1" />
-    <limit effort="100" lower="-1.570796327" upper="1.570796327" velocity="5"/>
+    <limit effort="100" lower="${-M_PI/2}" upper="${M_PI/2}" velocity="5"/>
     </joint>
     <link name="${name}_thumb_2_link">
@@ -260,12 +344,33 @@
           <mesh filename="package://schunk_description/meshes/sdh/finger.stl" />
         </geometry>
-        <material name="Schunk/LightGrey" />
-      </visual>
-      <collision>
-        <origin xyz="0 0 0" rpy="0 0 0" />
-        <geometry>
-          <mesh filename="package://schunk_description/meshes/sdh/finger.stl"/>
-        </geometry>
-      </collision>
+        <material name="Schunk/DarkGrey" />
+      </visual>
+      <collision>
+        <origin xyz="0 0 0" rpy="0 0 0" />
+        <geometry>
+          <mesh filename="package://schunk_description/meshes/sdh/finger.stl"/>
+        </geometry>
+      </collision>
+    </link>
+    <joint name="${name}_thumb_sensor_joint" type="fixed">
+      <origin xyz="0.01529 -0.011 ${0.01875+0.05}" rpy="-${M_PI/2} 0 ${M_PI/2}" />
+      <parent link="${name}_thumb_2_link"/>
+      <child link="${name}_thumb_sensor_link"/>
+    </joint>
+    <link name="${name}_thumb_sensor_link">
+      <xacro:default_inertial/>
+      <!--<visual>
+        <origin xyz="0 0 0" rpy="0 0 0" />
+        <geometry>
+          <mesh filename="package://schunk_description/meshes/sdh/finger.stl" />
+        </geometry>
+      <material name="Schunk/DarkGrey" />
+      </visual>
+      <collision>
+        <origin xyz="0 0 0" rpy="0 0 0" />
+        <geometry>
+          <mesh filename="package://schunk_description/meshes/sdh/finger.stl"/>
+        </geometry>
+      </collision>-->
     </link>
     <!-- joint between sdh_thumb_2_link and sdh_thumb_3_link -->
@@ -276,5 +381,5 @@
       <axis xyz="0 1 0" />
       <dynamics damping="1" />
-      <limit effort="100" lower="-1.570796327" upper="1.570796327" velocity="5"/>
+      <limit effort="100" lower="${-M_PI/2}" upper="${M_PI/2}" velocity="5"/>
     </joint>
     <link name="${name}_thumb_3_link">
@@ -285,5 +390,5 @@
           <mesh filename="package://schunk_description/meshes/sdh/finger_tip.stl" />
         </geometry>
-        <material name="Schunk/LightGrey" />
+        <material name="Schunk/DarkGrey" />
       </visual>
       <collision>
@@ -293,4 +398,25 @@
         </geometry>
       </collision>
+    </link>
+    <joint name="${name}_thumb_tip_sensor_joint" type="fixed">
+      <origin xyz="0.005151 -0.011 ${0.01943+0.05}" rpy="-${M_PI/2} 0 ${M_PI/2}" />
+      <parent link="${name}_thumb_3_link"/>
+      <child link="${name}_thumb_tip_sensor_link"/>
+    </joint>
+    <link name="${name}_thumb_tip_sensor_link">
+      <xacro:default_inertial/>
+      <!--<visual>
+        <origin xyz="0 0 0" rpy="0 0 0" />
+        <geometry>
+          <mesh filename="package://schunk_description/meshes/sdh/finger.stl" />
+        </geometry>
+      <material name="Schunk/DarkGrey" />
+      </visual>
+      <collision>
+        <origin xyz="0 0 0" rpy="0 0 0" />
+        <geometry>
+          <mesh filename="package://schunk_description/meshes/sdh/finger.stl"/>
+        </geometry>
+      </collision>-->
     </link>
     <!-- extensions -->
